File: kicad/pmod_optical.kicad_pcb (KiCad board)
At the start: 2 copper layers, 32 x 22 mm, 17 parts, among them IC1 SN74AHC126DR, J2 FCR684208R, J3 FCR684208T

Commit message: Added BOM
Parts:
- R1, R2, R3, R4, R5, R6, R7, R8: value 100K -> 100k

Commit message: Update BOM
Other:
- board text added: "Rev ${SchematicRevision}${PCBRevision}"
- board text removed: "Rev 2c"
