File: kicad/pmod_optical.kicad_sch (KiCad schematic)
At the start: 16 parts, among them IC1 SN74AHC126DR, J1 PMOD (6 Pin), J2 FCR684208R, J3 FCR684208T

Commit message: Added BOM
Parts:
- C1, C3, C4: Manufacturer_Name Johanson Technology Inc. -> (none); Manufacturer_Part_Number 250X15W104MV4E -> (none); Part (none) -> 0805 SMD Capacitor
- C2: Manufacturer_Name Johanson Technology Inc. -> (none); Manufacturer_Part_Number 251R15S300GV4E -> (none); Part (none) -> 0805 SMD Capacitor
- IC1: Part (none) -> SOIC SMD SN74AHC126DR; Vendor (none) -> Texas Instruments
- J1: Part (none) -> 1x6 0.1 Inch pitch right angle pin header
- J2: Part (none) -> FCR684208R; Vendor (none) -> Cliff Electronics Components
- J3: Part (none) -> FCR684208T; Vendor (none) -> Cliff Electronics Components
- R1, R2, R3, R4, R5, R6, R7, R8: value 100K -> 100k; Manufacturer_Name Panasonic -> (none); Manufacturer_Part_Number ERJ-P06F1003V -> (none); Part (none) -> 0805 SMD Resistor
Other:
- title: (none) -> PMOD_OPTICAL
Changed lines of the file:
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@@
 (kicad_sch (version 20230121) (generator eeschema)
   (paper "A4")
+  (title_block
+    (title "PMOD_OPTICAL")
+    (date "2023-07-27")
+    (rev "2c")
+  )
   (junction (at 133.35 85.09) (diameter 0) (color 0 0 0 0)
   )
@@
       (effects (font (size 1.27 1.27)) (justify left))
     )
-    (property "Value" "100K" (at 68.58 58.42 0)
+    (property "Value" "100k" (at 68.58 58.42 0)
       (effects (font (size 1.27 1.27)) (justify left))
     )
@@
       (effects (font (size 1.27 1.27)) hide)
     )
-    (property "Manufacturer_Name" "Panasonic" (at 71.12 57.15 0)
-      (effects (font (size 1.27 1.27)) hide)
-    )
-    (property "Manufacturer_Part_Number" "ERJ-P06F1003V" (at 71.12 57.15 0)
+    (property "Part" "0805 SMD Resistor" (at 71.12 57.15 0)
+      (effects (font (size 1.27 1.27)) hide)
+    )
+    (property "Vendor" "" (at 71.12 57.15 0)
       (effects (font (size 1.27 1.27)) hide)
     )
@@
       (effects (font (size 1.27 1.27)) hide)
     )
-    (property "Manufacturer_Name" "Johanson Technology Inc." (at 181.61 48.26 0)
-      (effects (font (size 1.27 1.27)) hide)
-    )
-    (property "Manufacturer_Part_Number" "251R15S300GV4E" (at 181.61 48.26 0)
+    (property "Part" "0805 SMD Capacitor" (at 181.61 48.26 0)
+      (effects (font (size 1.27 1.27)) hide)
+    )
+    (property "Vendor" "" (at 181.61 48.26 0)
       (effects (font (size 1.27 1.27)) hide)
     )
@@
       (effects (font (size 1.27 1.27)) hide)
     )
-    (property "Manufacturer_Name" "Johanson Technology Inc." (at 195.58 48.26 0)
-      (effects (font (size 1.27 1.27)) hide)
-    )
-    (property "Manufacturer_Part_Number" "250X15W104MV4E" (at 195.58 48.26 0)
+    (property "Part" "0805 SMD Capacitor" (at 195.58 48.26 0)
+      (effects (font (size 1.27 1.27)) hide)
+    )
+    (property "Vendor" "" (at 195.58 48.26 0)
       (effects (font (size 1.27 1.27)) hide)
     )
@@
       (effects (font (size 1.27 1.27)) hide)
     )
-    (property "Manufacturer_Name" "Johanson Technology Inc." (at 120.65 52.07 0)
-      (effects (font (size 1.27 1.27)) hide)
-    )
-    (property "Manufacturer_Part_Number" "250X15W104MV4E" (at 120.65 52.07 0)
+    (property "Part" "0805 SMD Capacitor" (at 120.65 52.07 0)
+      (effects (font (size 1.27 1.27)) hide)
+    )
+    (property "Vendor" "" (at 120.65 52.07 0)
       (effects (font (size 1.27 1.27)) hide)
     )
@@
       (effects (font (size 1.27 1.27)) (justify left))
     )
-    (property "Value" "100K" (at 140.97 68.58 0)
+    (property "Value" "100k" (at 140.97 68.58 0)
       (effects (font (size 1.27 1.27)) (justify left))
     )
@@
       (effects (font (size 1.27 1.27)) hide)
     )
-    (property "Manufacturer_Name" "Panasonic" (at 143.51 67.31 0)
-      (effects (font (size 1.27 1.27)) hide)
-    )
-    (property "Manufacturer_Part_Number" "ERJ-P06F1003V" (at 143.51 67.31 0)
+    (property "Part" "0805 SMD Resistor" (at 143.51 67.31 0)
+      (effects (font (size 1.27 1.27)) hide)
+    )
+    (property "Vendor" "" (at 143.51 67.31 0)
       (effects (font (size 1.27 1.27)) hide)
     )
@@
       (effects (font (size 1.27 1.27)) (justify left))
     )
-    (property "Value" "100K" (at 78.74 58.42 0)
+    (property "Value" "100k" (at 78.74 58.42 0)
       (effects (font (size 1.27 1.27)) (justify left))
     )
@@
       (effects (font (size 1.27 1.27)) hide)
     )
-    (property "Manufacturer_Name" "Panasonic" (at 81.28 57.15 0)
-      (effects (font (size 1.27 1.27)) hide)
-    )
-    (property "Manufacturer_Part_Number" "ERJ-P06F1003V" (at 81.28 57.15 0)
+    (property "Part" "0805 SMD Resistor" (at 81.28 57.15 0)
+      (effects (font (size 1.27 1.27)) hide)
+    )
+    (property "Vendor" "" (at 81.28 57.15 0)
       (effects (font (size 1.27 1.27)) hide)
     )
@@
       (effects (font (size 1.27 1.27)) (justify left))
     )
-    (property "Value" "100K" (at 71.12 68.58 0)
+    (property "Value" "100k" (at 71.12 68.58 0)
       (effects (font (size 1.27 1.27)) (justify left))
     )
@@
       (effects (font (size 1.27 1.27)) hide)
     )
-    (property "Manufacturer_Name" "Panasonic" (at 73.66 67.31 0)
-      (effects (font (size 1.27 1.27)) hide)
-    )
-    (property "Manufacturer_Part_Number" "ERJ-P06F1003V" (at 73.66 67.31 0)
+    (property "Part" "0805 SMD Resistor" (at 73.66 67.31 0)
+      (effects (font (size 1.27 1.27)) hide)
+    )
+    (property "Vendor" "" (at 73.66 67.31 0)
       (effects (font (size 1.27 1.27)) hide)
     )
@@
       (effects (font (size 1.27 1.27)) (justify left))
     )
-    (property "Value" "100K" (at 128.27 58.42 0)
+    (property "Value" "100k" (at 128.27 58.42 0)
       (effects (font (size 1.27 1.27)) (justify left))
     )
@@
       (effects (font (size 1.27 1.27)) hide)
     )
-    (property "Manufacturer_Name" "Panasonic" (at 130.81 57.15 0)
-      (effects (font (size 1.27 1.27)) hide)
-    )
-    (property "Manufacturer_Part_Number" "ERJ-P06F1003V" (at 130.81 57.15 0)
+    (property "Part" "0805 SMD Resistor" (at 130.81 57.15 0)
+      (effects (font (size 1.27 1.27)) hide)
+    )
+    (property "Vendor" "" (at 130.81 57.15 0)
       (effects (font (size 1.27 1.27)) hide)
     )
@@
       (effects (font (size 1.27 1.27)) (justify left) hide)
     )
+    (property "Part" "1x6 0.1 Inch pitch right angle pin header" (at 41.91 30.48 0)
+      (effects (font (size 1.27 1.27)) hide)
+    )
+    (property "Vendor" "" (at 41.91 30.48 0)
+      (effects (font (size 1.27 1.27)) hide)
+    )
     (pin "1")
     (pin "2")
@@
       (effects (font (size 1.27 1.27)) (justify left) hide)
     )
+    (property "Part" "FCR684208R" (at 217.17 40.64 0)
+      (effects (font (size 1.27 1.27)) hide)
+    )
+    (property "Vendor" "Cliff Electronics Components" (at 217.17 40.64 0)
+      (effects (font (size 1.27 1.27)) hide)
+    )
     (pin "1")
     (pin "2")
@@
       (effects (font (size 1.27 1.27)) (justify left))
     )
-    (property "Value" "100K" (at 138.43 58.42 0)
+    (property "Value" "100k" (at 138.43 58.42 0)
       (effects (font (size 1.27 1.27)) (justify left))
     )
@@
       (effects (font (size 1.27 1.27)) hide)
     )
-    (property "Manufacturer_Name" "Panasonic" (at 140.97 57.15 0)
-      (effects (font (size 1.27 1.27)) hide)
-    )
-    (property "Manufacturer_Part_Number" "ERJ-P06F1003V" (at 140.97 57.15 0)
+    (property "Part" "0805 SMD Resistor" (at 140.97 57.15 0)
+      (effects (font (size 1.27 1.27)) hide)
+    )
+    (property "Vendor" "" (at 140.97 57.15 0)
       (effects (font (size 1.27 1.27)) hide)
     )
@@
     (property "Datasheet" "https://www.ti.com/lit/gpn/SN74AHC126" (at 85.09 97.79 0)
       (effects (font (size 1.27 1.27)) (justify left) hide)
+    )
+    (property "Part" "SOIC SMD SN74AHC126DR" (at 91.44 77.47 0)
+      (effects (font (size 1.27 1.27)) hide)
+    )
+    (property "Vendor" "Texas Instruments" (at 91.44 77.47 0)
+      (effects (font (size 1.27 1.27)) hide)
     )
     (pin "1")
@@
       (effects (font (size 1.27 1.27)) (justify left))
     )
-    (property "Value" "100K" (at 130.81 68.58 0)
+    (property "Value" "100k" (at 130.81 68.58 0)
       (effects (font (size 1.27 1.27)) (justify left))
     )
@@
       (effects (font (size 1.27 1.27)) hide)
     )
-    (property "Manufacturer_Name" "Panasonic" (at 133.35 67.31 0)
-      (effects (font (size 1.27 1.27)) hide)
-    )
-    (property "Manufacturer_Part_Number" "ERJ-P06F1003V" (at 133.35 67.31 0)
+    (property "Part" "0805 SMD Resistor" (at 133.35 67.31 0)
+      (effects (font (size 1.27 1.27)) hide)
+    )
+    (property "Vendor" "" (at 133.35 67.31 0)
       (effects (font (size 1.27 1.27)) hide)
     )
@@
       (effects (font (size 1.27 1.27)) (justify left) hide)
     )
+    (property "Part" "FCR684208T" (at 218.44 99.06 0)
+      (effects (font (size 1.27 1.27)) hide)
+    )
+    (property "Vendor" "Cliff Electronics Components" (at 218.44 99.06 0)
+      (effects (font (size 1.27 1.27)) hide)
+    )
     (pin "1")
     (pin "2")
@@
       (effects (font (size 1.27 1.27)) (justify left))
     )
-    (property "Value" "100K" (at 81.28 68.58 0)
+    (property "Value" "100k" (at 81.28 68.58 0)
       (effects (font (size 1.27 1.27)) (justify left))
     )
@@
       (effects (font (size 1.27 1.27)) hide)
     )
-    (property "Manufacturer_Name" "Panasonic" (at 83.82 67.31 0)
-      (effects (font (size 1.27 1.27)) hide)
-    )
-    (property "Manufacturer_Part_Number" "ERJ-P06F1003V" (at 83.82 67.31 0)
+    (property "Part" "0805 SMD Resistor" (at 83.82 67.31 0)
+      (effects (font (size 1.27 1.27)) hide)
+    )
+    (property "Vendor" "" (at 83.82 67.31 0)
       (effects (font (size 1.27 1.27)) hide)
     )
@@
       (effects (font (size 1.27 1.27)) hide)
     )
-    (property "Manufacturer_Name" "Johanson Technology Inc." (at 195.58 92.71 0)
-      (effects (font (size 1.27 1.27)) hide)
-    )
-    (property "Manufacturer_Part_Number" "250X15W104MV4E" (at 195.58 92.71 0)
-      (effects (font (size 1.27 1.27)) hide)
-    )
+    (property "Part" "0805 SMD Capacitor" (at 195.58 92.71 0)
+      (effects (font (size 1.27 1.27)) hide)
+    )
+    (property "Vendor" "" (at 195.58 92.71 0)
+      (effects (font (size 1.27 1.27)) hide)
+    )

Commit message: Update BOM
Parts:
- C1, C3, C4: MPN (none) -> 0.1uF 0805 SMD Capacitor; Part 0805 SMD Capacitor -> (none)
- C2: MPN (none) -> 30pf 0805 SMD Capacitor; Part 0805 SMD Capacitor -> (none)
- IC1: MPN (none) -> SN74AHC126DR; Manufacturer (none) -> Texas Instruments; Notes (none) -> SOIC SMD SN74AHC126DR; Part SOIC SMD SN74AHC126DR -> (none); Vendor Texas Instruments -> (none)
- J1: MPN (none) -> TSW-106-08-L-S-RA; Manufacturer (none) -> Samtec; Notes (none) -> 1x6 0.1 Inch pitch right angle pin header; Part 1x6 0.1 Inch pitch right angle pin header -> (none)
- J2: MPN (none) -> FCR684208R; Manufacturer (none) -> Cliff Electronics Components; Part FCR684208R -> (none); Vendor Cliff Electronics Components -> (none)
- J3: MPN (none) -> FCR684208T; Manufacturer (none) -> Cliff Electronics Components; Part FCR684208T -> (none); Vendor Cliff Electronics Components -> (none)
- R1, R2, R3, R4, R5, R6, R7, R8: MPN (none) -> 100k ohm 0805 SMD Resistor; Part 0805 SMD Resistor -> (none)
Changed lines of the file:
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@@
     (title "PMOD_OPTICAL")
     (date "2023-07-27")
-    (rev "2c")
+    (rev "${SchematicRevision}")
   )
   (junction (at 133.35 85.09) (diameter 0) (color 0 0 0 0)
@@
       (effects (font (size 1.27 1.27)) hide)
     )
-    (property "Part" "0805 SMD Resistor" (at 71.12 57.15 0)
-      (effects (font (size 1.27 1.27)) hide)
-    )
-    (property "Vendor" "" (at 71.12 57.15 0)
+    (property "MPN" "100k ohm 0805 SMD Resistor" (at 71.12 57.15 0)
+      (effects (font (size 1.27 1.27)) hide)
+    )
+    (property "Manufacturer" "" (at 71.12 57.15 0)
+      (effects (font (size 1.27 1.27)) hide)
+    )
+    (property "Notes" "" (at 71.12 57.15 0)
       (effects (font (size 1.27 1.27)) hide)
     )
@@
       (effects (font (size 1.27 1.27)) hide)
     )
-    (property "Part" "0805 SMD Capacitor" (at 181.61 48.26 0)
-      (effects (font (size 1.27 1.27)) hide)
-    )
-    (property "Vendor" "" (at 181.61 48.26 0)
+    (property "MPN" "30pf 0805 SMD Capacitor" (at 181.61 48.26 0)
+      (effects (font (size 1.27 1.27)) hide)
+    )
+    (property "Manufacturer" "" (at 181.61 48.26 0)
+      (effects (font (size 1.27 1.27)) hide)
+    )
+    (property "Notes" "" (at 181.61 48.26 0)
       (effects (font (size 1.27 1.27)) hide)
     )
@@
       (effects (font (size 1.27 1.27)) hide)
     )
-    (property "Part" "0805 SMD Capacitor" (at 195.58 48.26 0)
-      (effects (font (size 1.27 1.27)) hide)
-    )
-    (property "Vendor" "" (at 195.58 48.26 0)
+    (property "MPN" "0.1uF 0805 SMD Capacitor" (at 195.58 48.26 0)
+      (effects (font (size 1.27 1.27)) hide)
+    )
+    (property "Manufacturer" "" (at 195.58 48.26 0)
+      (effects (font (size 1.27 1.27)) hide)
+    )
+    (property "Notes" "" (at 195.58 48.26 0)
       (effects (font (size 1.27 1.27)) hide)
     )
@@
       (effects (font (size 1.27 1.27)) hide)
     )
-    (property "Part" "0805 SMD Capacitor" (at 120.65 52.07 0)
-      (effects (font (size 1.27 1.27)) hide)
-    )
-    (property "Vendor" "" (at 120.65 52.07 0)
+    (property "MPN" "0.1uF 0805 SMD Capacitor" (at 120.65 52.07 0)
+      (effects (font (size 1.27 1.27)) hide)
+    )
+    (property "Manufacturer" "" (at 120.65 52.07 0)
+      (effects (font (size 1.27 1.27)) hide)
+    )
+    (property "Notes" "" (at 120.65 52.07 0)
       (effects (font (size 1.27 1.27)) hide)
     )
@@
       (effects (font (size 1.27 1.27)) hide)
     )
-    (property "Part" "0805 SMD Resistor" (at 143.51 67.31 0)
-      (effects (font (size 1.27 1.27)) hide)
-    )
-    (property "Vendor" "" (at 143.51 67.31 0)
+    (property "MPN" "100k ohm 0805 SMD Resistor" (at 143.51 67.31 0)
+      (effects (font (size 1.27 1.27)) hide)
+    )
+    (property "Manufacturer" "" (at 143.51 67.31 0)
+      (effects (font (size 1.27 1.27)) hide)
+    )
+    (property "Notes" "" (at 143.51 67.31 0)
       (effects (font (size 1.27 1.27)) hide)
     )
@@
       (effects (font (size 1.27 1.27)) hide)
     )
-    (property "Part" "0805 SMD Resistor" (at 81.28 57.15 0)
-      (effects (font (size 1.27 1.27)) hide)
-    )
-    (property "Vendor" "" (at 81.28 57.15 0)
+    (property "MPN" "100k ohm 0805 SMD Resistor" (at 81.28 57.15 0)
+      (effects (font (size 1.27 1.27)) hide)
+    )
+    (property "Manufacturer" "" (at 81.28 57.15 0)
+      (effects (font (size 1.27 1.27)) hide)
+    )
+    (property "Notes" "" (at 81.28 57.15 0)
       (effects (font (size 1.27 1.27)) hide)
     )
@@
       (effects (font (size 1.27 1.27)) hide)
     )
-    (property "Part" "0805 SMD Resistor" (at 73.66 67.31 0)
-      (effects (font (size 1.27 1.27)) hide)
-    )
-    (property "Vendor" "" (at 73.66 67.31 0)
+    (property "MPN" "100k ohm 0805 SMD Resistor" (at 73.66 67.31 0)
+      (effects (font (size 1.27 1.27)) hide)
+    )
+    (property "Manufacturer" "" (at 73.66 67.31 0)
+      (effects (font (size 1.27 1.27)) hide)
+    )
+    (property "Notes" "" (at 73.66 67.31 0)
       (effects (font (size 1.27 1.27)) hide)
     )
@@
       (effects (font (size 1.27 1.27)) hide)
     )
-    (property "Part" "0805 SMD Resistor" (at 130.81 57.15 0)
-      (effects (font (size 1.27 1.27)) hide)
-    )
-    (property "Vendor" "" (at 130.81 57.15 0)
+    (property "MPN" "100k ohm 0805 SMD Resistor" (at 130.81 57.15 0)
+      (effects (font (size 1.27 1.27)) hide)
+    )
+    (property "Manufacturer" "" (at 130.81 57.15 0)
+      (effects (font (size 1.27 1.27)) hide)
+    )
+    (property "Notes" "" (at 130.81 57.15 0)
       (effects (font (size 1.27 1.27)) hide)
     )
@@
       (effects (font (size 1.27 1.27)) (justify left) hide)
     )
-    (property "Datasheet" "" (at 25.4 30.48 0)
+    (property "Datasheet" "https://suddendocs.samtec.com/catalog_english/tsw_th.pdf)" (at 25.4 30.48 0)
       (effects (font (size 1.27 1.27)) (justify left) hide)
     )
-    (property "Part" "1x6 0.1 Inch pitch right angle pin header" (at 41.91 30.48 0)
-      (effects (font (size 1.27 1.27)) hide)
-    )
-    (property "Vendor" "" (at 41.91 30.48 0)
+    (property "MPN" "TSW-106-08-L-S-RA" (at 41.91 30.48 0)
+      (effects (font (size 1.27 1.27)) hide)
+    )
+    (property "Manufacturer" "Samtec" (at 41.91 30.48 0)
+      (effects (font (size 1.27 1.27)) hide)
+    )
+    (property "Notes" "1x6 0.1 Inch pitch right angle pin header" (at 41.91 30.48 0)
       (effects (font (size 1.27 1.27)) hide)
     )
@@
       (effects (font (size 1.27 1.27)) (justify left) hide)
     )
-    (property "Part" "FCR684208R" (at 217.17 40.64 0)
-      (effects (font (size 1.27 1.27)) hide)
-    )
-    (property "Vendor" "Cliff Electronics Components" (at 217.17 40.64 0)
+    (property "MPN" "FCR684208R" (at 217.17 40.64 0)
+      (effects (font (size 1.27 1.27)) hide)
+    )
+    (property "Manufacturer" "Cliff Electronics Components" (at 217.17 40.64 0)
+      (effects (font (size 1.27 1.27)) hide)
+    )
+    (property "Notes" "" (at 217.17 40.64 0)
       (effects (font (size 1.27 1.27)) hide)
     )
@@
       (effects (font (size 1.27 1.27)) hide)
     )
-    (property "Part" "0805 SMD Resistor" (at 140.97 57.15 0)
-      (effects (font (size 1.27 1.27)) hide)
-    )
-    (property "Vendor" "" (at 140.97 57.15 0)
+    (property "MPN" "100k ohm 0805 SMD Resistor" (at 140.97 57.15 0)
+      (effects (font (size 1.27 1.27)) hide)
+    )
+    (property "Manufacturer" "" (at 140.97 57.15 0)
+      (effects (font (size 1.27 1.27)) hide)
+    )
+    (property "Notes" "" (at 140.97 57.15 0)
       (effects (font (size 1.27 1.27)) hide)
     )
@@
       (effects (font (size 1.27 1.27)) (justify left) hide)
     )
-    (property "Part" "SOIC SMD SN74AHC126DR" (at 91.44 77.47 0)
-      (effects (font (size 1.27 1.27)) hide)
-    )
-    (property "Vendor" "Texas Instruments" (at 91.44 77.47 0)
+    (property "MPN" "SN74AHC126DR" (at 91.44 77.47 0)
+      (effects (font (size 1.27 1.27)) hide)
+    )
+    (property "Manufacturer" "Texas Instruments" (at 91.44 77.47 0)
+      (effects (font (size 1.27 1.27)) hide)
+    )
+    (property "Notes" "SOIC SMD SN74AHC126DR" (at 91.44 77.47 0)
       (effects (font (size 1.27 1.27)) hide)
     )
@@
       (effects (font (size 1.27 1.27)) hide)
     )
-    (property "Part" "0805 SMD Resistor" (at 133.35 67.31 0)
-      (effects (font (size 1.27 1.27)) hide)
-    )
-    (property "Vendor" "" (at 133.35 67.31 0)
+    (property "MPN" "100k ohm 0805 SMD Resistor" (at 133.35 67.31 0)
+      (effects (font (size 1.27 1.27)) hide)
+    )
+    (property "Manufacturer" "" (at 133.35 67.31 0)
+      (effects (font (size 1.27 1.27)) hide)
+    )
+    (property "Notes" "" (at 133.35 67.31 0)
       (effects (font (size 1.27 1.27)) hide)
     )
@@
       (effects (font (size 1.27 1.27)) (justify left) hide)
     )
-    (property "Part" "FCR684208T" (at 218.44 99.06 0)
-      (effects (font (size 1.27 1.27)) hide)
-    )
-    (property "Vendor" "Cliff Electronics Components" (at 218.44 99.06 0)
+    (property "MPN" "FCR684208T" (at 218.44 99.06 0)
+      (effects (font (size 1.27 1.27)) hide)
+    )
+    (property "Manufacturer" "Cliff Electronics Components" (at 218.44 99.06 0)
+      (effects (font (size 1.27 1.27)) hide)
+    )
+    (property "Notes" "" (at 218.44 99.06 0)
       (effects (font (size 1.27 1.27)) hide)
     )
@@
       (effects (font (size 1.27 1.27)) hide)
     )
-    (property "Part" "0805 SMD Resistor" (at 83.82 67.31 0)
-      (effects (font (size 1.27 1.27)) hide)
-    )
-    (property "Vendor" "" (at 83.82 67.31 0)
+    (property "MPN" "100k ohm 0805 SMD Resistor" (at 83.82 67.31 0)
+      (effects (font (size 1.27 1.27)) hide)
+    )
+    (property "Manufacturer" "" (at 83.82 67.31 0)
+      (effects (font (size 1.27 1.27)) hide)
+    )
+    (property "Notes" "" (at 83.82 67.31 0)
       (effects (font (size 1.27 1.27)) hide)
     )
@@
       (effects (font (size 1.27 1.27)) hide)
     )
-    (property "Part" "0805 SMD Capacitor" (at 195.58 92.71 0)
-      (effects (font (size 1.27 1.27)) hide)
-    )
-    (property "Vendor" "" (at 195.58 92.71 0)
-      (effects (font (size 1.27 1.27)) hide)
-    )
+    (property "MPN" "0.1uF 0805 SMD Capacitor" (at 195.58 92.71 0)
+      (effects (font (size 1.27 1.27)) hide)
+    )
+    (property "Manufacturer" "" (at 195.58 92.71 0)
+      (effects (font (size 1.27 1.27)) hide)
+    )
+    (property "Notes" "" (at 195.58 92.71 0)
+      (effects (font (size 1.27 1.27)) hide)
+    )
